File: hardware/main_board.brd (EAGLE design)
At the start: 109.9 x 68.6 mm, 113 parts, among them IC1 IC_USBLC6-2, IC2 LM1117IMPX-3.3, IC3 PIC32MX795F512, IC4 ENC28J60, IC5 LM1117MPX-2.5, U1 USD-SOCKETUSD, U2 VS1003, X2 CRYSTALS-NOGND-CFPX-217, X3 KUSBVX, Y1 CRYSTAL-GROUNDEDSMD-5X3.2, Y2 CRYSTAL-GROUNDEDSMD-5X3.2, Y3 CRYSTAL-GROUNDEDSMD-5X3.2

Commit message: PCB updated
Parts:
- removed R14: (no value), rcl:R1206
- C38: device rcl:C0603 -> rcl:C0402
- moved R9 4.89 mm to (54.3, 52.3), turned to 0 degrees
- moved C38 4.08 mm to (48.2, 47.7), turned to 180 degrees
- moved C28 2.67 mm to (49.4, 52.3)
- moved JP2 2.56 mm to (47.1, 54.8)
- moved C12 2.54 mm to (44.9, 60.5)
- moved F1 2.54 mm to (48.9, 61.9)
- moved C11 2.05 mm to (56.7, 45.5), turned to 270 degrees
- moved C15 1.96 mm to (66.7, 61.3)
- moved Y1 0.64 mm to (50.5, 20.8)
- moved C52 0.64 mm to (66.7, 53.9)
- moved C1 0.63 mm to (51.4, 16.8)
- moved C2 0.63 mm to (49.7, 16.8)
- moved R18 0.63 mm to (43.2, 47.0)
Connections:
- net RG7 renamed RG7_SDA2A
- net RG8 renamed RG8_SCL2A
- removed net 3V_IN: C14.1, C15.+, C18.1, C19.1, C25.1, C26.+, C29.1, C31.1, C32.1, C40.1, C41.1, C42.1, C56.1, IC2.2, IC2.TAB, IC4.P$15, IC4.P$19, IC4.P$20, IC4.P$25, IC4.P$28, JP3.4, L3.1, R11.2, R13.2, R14.1, R30.2, R8.2, SV1.33, SV1.34, U$2.3, U$2.7, U$2.8, U1.4, U2.14, U2.19, U2.32, U2.6
- net 3V: now also C14.1, C15.+, C18.1, C19.1, C25.1, C26.+, C29.1, C31.1, C32.1, C40.1, C41.1, C42.1, C56.1, IC2.2, IC2.TAB, IC4.P$15, IC4.P$19, IC4.P$20, IC4.P$25, IC4.P$28, JP3.4, L3.1, R11.2, R13.2, R30.2, R8.2, SV1.33, SV1.34, U$2.3, U$2.7, U$2.8, U1.4, U2.14, U2.19, U2.32, U2.6; no longer R14.2
Routing:
- net 3V: track 101.3 -> 443.9 mm, vias 0 -> 9
- net 3V_IN: track 335.7 -> 0.00 mm, vias 6 -> 0
- net VBUS: track 192.5 -> 190.0 mm
- net N$17: track 1.92 -> 4.26 mm
- net OSC2: track 17.7 -> 17.0 mm
- net AN_3V: track 10.5 -> 9.83 mm
- net OSC1: track 17.6 -> 17.0 mm
- net GND: track 59.2 -> 58.7 mm
